File: NovaDrone/Half_Bridge.kicad_sch (KiCad schematic)
At the start: 13 parts, among them Q4 SQJA06EP-T1_GE3, U1 INA181A1IDBVR

Commit message: PCB temperature measurement
Parts:
- renumbered Q to Q3
Changed lines of the file:
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@@
 		(dnp no)
 		(fields_autoplaced yes)
-		(property "Reference" "Q"
+		(property "Reference" "Q?"
 			(at 120.65 59.6899 0)
 			(effects
@@
 					(unit 1)
 				)
+				(path "/7036a814-0f41-4c6c-a077-a78d90a22423/60c9f1ab-8310-4b41-87cd-18a1725e670c"
+					(reference "Q?")
+					(unit 1)
+				)

Commit message: Interfaces Update
Parts:
- added C21: 1uF 50V, Capacitor_SMD:C_0805_2012Metric, symbol Device:C
- C1: value 0.1uF -> 0.1uF 50V
Connections:
- net Power_GND: now also C21.2
- net at Q4.5: now also C21.1
Changed lines of the file:
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@@
 	(generator "eeschema")
 	(generator_version "9.0")
-	(paper "A2")
+	(paper "A5")
 	(title_block
 		(title "NovaDrone")
@@
 	)
 	(junction
+		(at 116.84 24.13)
+		(diameter 0)
+		(color 0 0 0 0)
+	)
+	(junction
 		(at 116.84 86.36)
 		(diameter 0)
@@
 	(wire
 		(pts
+			(xy 116.84 24.13) (xy 116.84 30.48)
+		)
+		(stroke
+			(width 0)
+			(type default)
+		)
+	)
+	(wire
+		(pts
 			(xy 107.95 38.1) (xy 107.95 35.56)
 		)
@@
 	(wire
 		(pts
+			(xy 124.46 24.13) (xy 116.84 24.13)
+		)
+		(stroke
+			(width 0)
+			(type default)
+		)
+	)
+	(wire
+		(pts
+			(xy 139.7 26.67) (xy 139.7 24.13)
+		)
+		(stroke
+			(width 0)
+			(type default)
+		)
+	)
+	(wire
+		(pts
 			(xy 93.98 60.96) (xy 93.98 69.85)
 		)
@@
 	(wire
 		(pts
-			(xy 116.84 26.67) (xy 116.84 30.48)
+			(xy 116.84 20.32) (xy 116.84 24.13)
 		)
 		(stroke
@@
 		(pts
 			(xy 107.95 35.56) (xy 110.49 35.56)
+		)
+		(stroke
+			(width 0)
+			(type default)
+		)
+	)
+	(wire
+		(pts
+			(xy 139.7 24.13) (xy 132.08 24.13)
 		)
 		(stroke
@@
 	)
 	(symbol
+		(lib_id "Device:C")
+		(at 128.27 24.13 90)
+		(mirror x)
+		(unit 1)
+		(exclude_from_sim no)
+		(in_bom yes)
+		(on_board yes)
+		(dnp no)
+		(property "Reference" "C21"
+			(at 128.016 20.32 90)
+			(effects
+				(font
+					(size 1.27 1.27)
+				)
+			)
+		)
+		(property "Value" "1uF 50V"
+			(at 128.27 28.194 90)
+			(effects
+				(font
+					(size 1.27 1.27)
+				)
+			)
+		)
+		(property "Footprint" "Capacitor_SMD:C_0805_2012Metric"
+			(at 132.08 25.0952 0)
+			(effects
+				(font
+					(size 1.27 1.27)
+				)
+				(hide yes)
+			)
+		)
+		(property "Datasheet" "https://www.mouser.fr/datasheet/2/585/MLCC-1837944.pdf"
+			(at 128.27 24.13 0)
+			(effects
+				(font
+					(size 1.27 1.27)
+				)
+				(hide yes)
+			)
+		)
+		(property "Description" "Multilayer Ceramic Capacitors MLCC - SMD/SMT 1uF+/-10% 50V X7R 2012"
+			(at 128.27 24.13 0)
+			(effects
+				(font
+					(size 1.27 1.27)
+				)
+				(hide yes)
+			)
+		)
+		(property "Manufacturer_Name" "Samsung Electro-Mechanics"
+			(at 128.27 24.13 0)
+			(effects
+				(font
+					(size 1.27 1.27)
+				)
+				(hide yes)
+			)
+		)
+		(property "Manufacturer_Part_Number" " CL21B105KBFNNNE"
+			(at 128.27 24.13 0)
+			(effects
+				(font
+					(size 1.27 1.27)
+				)
+				(hide yes)
+			)
+		)
+		(property "Packaging" " 0805 (2012 mm)"
+			(at 128.27 24.13 0)
+			(effects
+				(font
+					(size 1.27 1.27)
+				)
+				(hide yes)
+			)
+		)
+		(pin "1"
+		)
+		(pin "2"
+		)
+		(instances
+			(project "NovaDrone"
+				(path "/7036a814-0f41-4c6c-a077-a78d90a22423/3d63b6fa-9b75-44ef-b487-19f1bfbe12f4"
+					(reference "C23")
+					(unit 1)
+				)
+				(path "/7036a814-0f41-4c6c-a077-a78d90a22423/60c9f1ab-8310-4b41-87cd-18a1725e670c"
+					(reference "C21")
+					(unit 1)
+				)
+				(path "/7036a814-0f41-4c6c-a077-a78d90a22423/f138b3a8-ec69-4954-8088-e3c29779a6aa"
+					(reference "C22")
+					(unit 1)
+				)
+			)
+		)
+	)
+	(symbol
 		(lib_id "BassingaLib_Mosfets:SQJA06EP-T1_GE3")
 		(at 116.84 35.56 0)
@@
 	(symbol
 		(lib_id "BassingaLib_Power_Symbols:Power")
-		(at 116.84 25.4 0)
+		(at 116.84 19.05 0)
 		(unit 1)
 		(exclude_from_sim no)
@@
 		(dnp no)
 		(property "Reference" "#PWR01"
-			(at 116.84 21.844 0)
+			(at 116.84 15.494 0)
 			(effects
 				(font
@@
 		)
 		(property "Value" "6S_Power"
-			(at 116.84 22.86 0)
+			(at 116.84 16.51 0)
 			(effects
 				(font
@@
 		)
 		(property "Footprint" ""
-			(at 116.84 25.4 0)
+			(at 116.84 19.05 0)
 			(effects
 				(font
@@
 		)
 		(property "Datasheet" ""
-			(at 116.84 25.4 0)
+			(at 116.84 19.05 0)
 			(effects
 				(font
@@
 		)
 		(property "Description" ""
-			(at 116.84 25.4 0)
+			(at 116.84 19.05 0)
 			(effects
 				(font
@@
 			)
 		)
-		(property "Value" "0.1uF"
+		(property "Value" "0.1uF 50V"
 			(at 162.56 71.374 90)
 			(effects
@@
 					(unit 1)
 				)
+			)
+		)
+	)
+	(symbol
+		(lib_id "BassingaLib_Power_Symbols:Power_GND")
+		(at 139.7 26.67 0)
+		(unit 1)
+		(exclude_from_sim no)
+		(in_bom no)
+		(on_board no)
+		(dnp no)
+		(fields_autoplaced yes)
+		(property "Reference" "#PWR061"
+			(at 139.7 32.258 0)
+			(effects
+				(font
+					(size 1.27 1.27)
+				)
+				(hide yes)
+			)
+		)
+		(property "Value" "Power_GND"
+			(at 139.7 31.75 0)
+			(effects
+				(font
+					(size 1.27 1.27)
+				)
+			)
+		)
+		(property "Footprint" ""
+			(at 139.7 26.67 0)
+			(effects
+				(font
+					(size 1.27 1.27)
+				)
+				(hide yes)
+			)
+		)
+		(property "Datasheet" ""
+			(at 139.7 26.67 0)
+			(effects
+				(font
+					(size 1.27 1.27)
+				)
+				(hide yes)
+			)
+		)
+		(property "Description" ""
+			(at 139.7 26.67 0)
+			(effects
+				(font
+					(size 1.27 1.27)
+				)
+				(hide yes)
+			)
+		)
+		(pin ""
+		)
+		(instances
+			(project "NovaDrone"
+				(path "/7036a814-0f41-4c6c-a077-a78d90a22423/3d63b6fa-9b75-44ef-b487-19f1bfbe12f4"
+					(reference "#PWR063")
+					(unit 1)
+				)
+				(path "/7036a814-0f41-4c6c-a077-a78d90a22423/60c9f1ab-8310-4b41-87cd-18a1725e670c"
+					(reference "#PWR061")
+					(unit 1)
+				)
+				(path "/7036a814-0f41-4c6c-a077-a78d90a22423/f138b3a8-ec69-4954-8088-e3c29779a6aa"
+					(reference "#PWR062")
+					(unit 1)
+				)
