File: NovaDrone/MCU.kicad_sch (KiCad schematic)
At the start: 1 part, among them IC4 STM32G473CCT3

Commit message: Interfaces Update
Parts:
- added C15, C16, C27, C31, C8: 0.1uF 50V, Capacitor_SMD:C_0603_1608Metric, symbol Device:C
- added C17: 4.7uF 50V, Capacitor_SMD:C_1206_3216Metric, symbol Device:C
- added C24, C26: 1uF 50V, Capacitor_SMD:C_0805_2012Metric, symbol Device:C
- added C25: 15nF, Capacitor_SMD:C_0603_1608Metric, symbol Device:C
- added C32, C33: 12nF 50V 5%, Capacitor_SMD:C_0603_1608Metric, symbol Device:C
- added LED1: BLUE, BassinaLib_LEDs:LEDM168X80N, symbol BassinaLib_LEDs:APHD1608LQBC_D
- added R41, R43: 10k 1%, Resistor_SMD:R_0603_1608Metric, symbol Device:R
- added R44: 680R 1%, Resistor_SMD:R_0603_1608Metric, symbol Device:R
- added Y1: ECS-80-10-30B-CWN-TR, BassinaLib_Crystals:ECS801830BAGNTR, symbol BassinaLib_Crystals:ECS-80-10-30B-CWN-TR
Connections:
- net OSC1: now also C33.2, Y1.1
- net OSC2: now also C32.2, Y1.3
- net nRST: now also C31.2, R43.2
- net GND: now reaches IC4.19 (VSSA)
- net GND: now also IC4.23 (VSS_1), IC4.35 (VSS_2), IC4.47 (VSS_3), C15.2, C16.1, C17.2, C24.1, C25.1, C26.1, C27.1, C31.1, C32.1, C33.1, C8.1, LED1.1 (K), R41.1, Y1.2, Y1.4
- net Vref: now reaches IC4.20 (VREF+)
- net Vref: now also C26.2, C27.2
- net +3.3V: now reaches IC4.21 (VDDA)
- net +3.3V: now also IC4.24 (VDD_1), IC4.36 (VDD_2), IC4.48 (VDD_3), C15.1, C16.2, C17.1, C24.2, C25.2, C8.2, R43.1
- net at IC4.25 (PB11): now also R44.1
- net FDCAN2_STB: now reaches IC4.41 (PB4)
- net at IC4.45 (PB8-BOOT0): now also R41.2
- new net: LED1.2 (A), R44.2
- no-connect marks 8 -> 7
Other:
- moved on the sheet: IC4

Commit message: Power Supply
Connections:
- net Vref is gone; now on net +3.3V: C26.2, C27.2, IC4.20 (VREF+)
- net V10_Mesure renamed V12_Mesure
