File: ESC/ESC.kicad_pcb (KiCad board)
At the start: 2 copper layers, 141 parts, among them IC1 TCAN3403DDFRQ1, IC2 UCC27211DR, IC3 UCC27211DR, IC4 UCC27211DR, IC5 STM32G473CCT3, IC6 BD433M5FP-CE2, J1 JST PH 4Pin, J2 JST SH 5Pin, J3 JST SH 3Pin, J4 MR30PW-M, J5 XT30PW-M, Q1 SQJA06EP-T1_GE3, Q2 SQJA06EP-T1_GE3, Q3 SQJA06EP-T1_GE3, Q4 SQJA06EP-T1_GE3, Q5 SQJA06EP-T1_GE3, Q6 SQJA06EP-T1_GE3, U1 INA181A1IDBVR, U2 INA181A1IDBVR, U3 INA181A1IDBVR, Y1 ECS-80-10-30B-CWN-TR

Commit message: PCB Layout Update
Parts:
- removed R51: 0R 1%, Resistor_SMD:R_0603_1608Metric
- C27, C28, C29, C3, C31, C32, C33, C34, C35, C36, C37, C38, C4, C40, C43, D2, IC1, IC5, IC6, LED1, R3, R45, R46, R47, Y1: moved to B.Cu
- moved C27 314.1 mm to (61.0, 95.2), turned to -90 degrees
- moved LED1 313.3 mm to (61.0, 103.0), turned to 180 degrees
- moved S1 310.0 mm to (45.2, 100.0), turned to 180 degrees
- moved R47 309.8 mm to (61.0, 104.8), turned to 180 degrees
- moved D2 309.1 mm to (35.5, 99.8), turned to 180 degrees
- moved J1 307.0 mm to (38.9, 102.8), turned to 90 degrees
- moved Y1 305.4 mm to (69.8, 85.0)
- moved C38 304.4 mm to (67.0, 102.8), turned to 180 degrees
- moved R46 304.1 mm to (67.0, 104.8), turned to 180 degrees
- moved R45 300.1 mm to (69.8, 81.2)
- moved C32 298.3 mm to (63.8, 93.0), turned to -90 degrees
- moved J3 297.2 mm to (53.5, 96.2), turned to 180 degrees
- moved C36 295.8 mm to (79.2, 99.5), turned to 90 degrees
- moved IC5 295.2 mm to (70.5, 96.5), turned to -90 degrees
- moved C28 294.0 mm to (68.2, 89.0)
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Connections:
- C15 pad 1: Power_GND -> GND
- C16 pad 1: Power_GND -> GND
- C17 pad 1: Power_GND -> GND
- C18 pad 2: Power_GND -> GND
- C20 pad 1: Power_GND -> GND
- C21 pad 2: Power_GND -> GND
- C23 pad 1: Power_GND -> GND
- C24 pad 2: Power_GND -> GND
- C26 pad 1: Power_GND -> GND
- C39 pad 1: Power_GND -> GND
- C41 pad 2: Power_GND -> GND
- C44 pad 2: Power_GND -> GND
- C45 pad 1: Power_GND -> GND
- D11 pad 2: Power_GND -> GND
- J5 pad N: Power_GND -> GND
- LED2 pad 1: Power_GND -> GND
- PS1 pad 4: Power_GND -> GND
- R27 pad 2: Power_GND -> GND
- R35 pad 2: Power_GND -> GND
- R43 pad 2: Power_GND -> GND
- U1 pad 4: Power_GND -> GND
- U2 pad 4: Power_GND -> GND
- U3 pad 4: Power_GND -> GND
Other:
- board outline added: 80 x 52.5 mm
- copper layers 2 -> 4

Commit message: Update 25.07.2025
Parts:
- C1, C2, C30, C5, D3, D4, R1, R16, R17, R2, R6, R7, R8, R9, TH1: moved to B.Cu
- LED1, R47: moved to F.Cu
- moved R9 136.9 mm to (34.5, 83.0), turned to -90 degrees
- moved R8 135.2 mm to (37.0, 83.8)
- moved D4 129.5 mm to (36.3, 86.5), turned to 180 degrees
- moved D1 122.5 mm to (65.0, 101.7), turned to -90 degrees
- moved R1 117.7 mm to (48.5, 78.0)
- moved R2 117.0 mm to (48.5, 76.2), turned to 180 degrees
- moved C1 112.3 mm to (63.2, 105.2), turned to 90 degrees
- moved R7 111.2 mm to (60.7, 76.8), turned to 180 degrees
- moved C2 109.1 mm to (65.5, 105.2), turned to 90 degrees
- moved R4 107.8 mm to (60.5, 93.2)
- moved R5 107.6 mm to (60.5, 95.0)
- moved R16 106.6 mm to (69.3, 76.5)
- moved D3 106.0 mm to (59.8, 79.8)
- moved C5 105.6 mm to (68.5, 106.0), turned to 180 degrees
- moved R17 105.6 mm to (69.3, 74.7), turned to 180 degrees
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Connections:
- net Net-(PS1-SW) renamed /Power_Supply/SW
- C47 pad 1: Net-(PS1-FB) -> GND
- C48 pad 1: Net-(PS1-FB) -> GND
Routing:
- net +12V: track 0.00 -> 20.8 mm
- net Net-(J3-Pad3): track 0.00 -> 14.9 mm
- net /MCU/UART2_RX: track 0.00 -> 10.3 mm
- net /MCU/UART2_TX: track 0.00 -> 7.22 mm
- net Net-(J3-Pad1): track 0.00 -> 7.02 mm
- net +22V: track 0.00 -> 6.09 mm
- net Net-(PS1-FB): track 0.00 -> 5.48 mm
- net Net-(PS1-BST): track 0.00 -> 2.06 mm
- net Net-(LED4-A): track 0.00 -> 2.00 mm
- net Net-(LED1-A): track 0.00 -> 1.95 mm
- net Net-(LED3-A): track 0.00 -> 1.88 mm
- net Net-(LED2-A): track 0.00 -> 1.88 mm
- added copper zone on F.Cu, net +12V
- added copper zone on F.Cu, net +22V
- added copper zone on F.Cu, net /Power_Supply/SW
- added copper zone on F.Cu, net GND
- added copper zone on In1.Cu, net GND
- added copper zone on In2.Cu, net GND
Other:
- board size 80 x 52.5 mm -> 80 x 55 mm

Commit message: PCB nearly completed
Parts:
- C19, C20, C22, C23, C25, C26, D10, D5, D6, D7, D8, D9, IC2, IC3, IC4, R21, R22, R23, R24, R25, R26, R27, R28, R29, R30, R31, R32, R33, R34, R35, R36, R37, R38, R39, R40, R41, R42, R43, R44, U1, U2, U3: moved to B.Cu
- moved U1 139.7 mm to (78.5, 70.9), turned to 180 degrees
- moved D6 134.2 mm to (84.8, 57.8)
- moved D5 133.9 mm to (84.8, 61.4)
- moved C18 130.3 mm to (89.9, 94.6), turned to -90 degrees
- moved R27 127.3 mm to (84.2, 67.5), turned to 90 degrees
- moved C19 127.0 mm to (78.0, 68.1)
- moved U3 119.1 mm to (78.5, 88.5), turned to 180 degrees
- moved U2 118.4 mm to (78.7, 105.6), turned to 180 degrees
- moved R25 115.9 mm to (89.8, 60.4), turned to 180 degrees
- moved R23 115.7 mm to (89.8, 57.0)
- moved R24 115.1 mm to (89.8, 65.9), turned to 180 degrees
- moved R26 115.1 mm to (89.9, 70.6)
- moved R21 115.1 mm to (89.8, 58.7)
- moved R22 114.9 mm to (89.8, 67.7), turned to 180 degrees
- moved D9 114.5 mm to (84.5, 79.1)
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Connections:
- C10 pad 2: /Phase_3 -> /Phase_2
- C14 pad 2: /Phase_2 -> /Phase_3
- D1 pad 1: /MCU/UART2_RX -> /MCU/UART2_TX
- D1 pad 2: /MCU/UART2_TX -> /MCU/UART2_RX
- IC5 pad 25: Net-(IC5-PB11) -> unconnected-(IC5-PB11-Pad25)
- IC5 pad 26: /Vbus_Mesure -> /Phase_3
- IC5 pad 27: /Phase_3 -> /V12_Mesure
- IC5 pad 28: /V12_Mesure -> /V3.3_Mesure
- IC5 pad 29: /V3.3_Mesure -> /Vbus_Mesure
- IC5 pad 33: unconnected-(IC5-PA11-Pad33) -> Net-(IC5-PA11)
- R11 pad 1: /OUT1 -> /OUT2
- R11 pad 2: /Phase_3 -> /Phase_2
- R13 pad 2: /Phase_3 -> /Phase_2
- R14 pad 1: /OUT1 -> /OUT3
- R14 pad 2: /Phase_2 -> /Phase_3
- R15 pad 2: /Phase_2 -> /Phase_3
- R47 pad 1: Net-(IC5-PB11) -> Net-(IC5-PA11)
Routing:
- net +3.3V: track 0.00 -> 168.8 mm, vias 0 -> 5
- net /OUT3: track 0.00 -> 50.6 mm, vias 0 -> 1
- net /OUT1: track 0.00 -> 45.2 mm, vias 0 -> 1
- net /Vbus_Mesure: track 0.00 -> 44.8 mm, vias 0 -> 2
- net /V3.3_Mesure: track 0.00 -> 39.5 mm, vias 0 -> 2
- net /OUT2: track 0.00 -> 37.1 mm, vias 0 -> 1
- net /V12_Mesure: track 0.00 -> 32.3 mm, vias 0 -> 2
- net /PCB_Temp: track 0.00 -> 28.9 mm
- net /MCU/nRST: track 0.00 -> 26.3 mm, vias 0 -> 1
- net /CANL: track 0.00 -> 26.2 mm, vias 0 -> 1
- net /MCU/FDCAN2_STB: track 0.00 -> 18.6 mm, vias 0 -> 2
- net /CANH: track 0.00 -> 18.2 mm, vias 0 -> 1
- net +22V: track 6.09 -> 23.8 mm, vias 0 -> 1
- net /MCU/FDCAN2_RX: track 0.00 -> 13.8 mm
- net /MCU/FDCAN2_TX: track 0.00 -> 13.2 mm
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- added copper zone on B.Cu, net GND

Commit message: End of Placement
Parts:
- C7: moved to B.Cu
- IC2, IC4: moved to F.Cu
- moved C13 77.9 mm to (99.9, 104.9), turned to 180 degrees
- moved C8 52.6 mm to (100.0, 96.7), turned to 180 degrees
- moved C12 47.4 mm to (68.3, 66.4)
- moved IC4 40.8 mm to (101.8, 100.7), turned to 0 degrees
- moved C11 32.8 mm to (100.2, 65.1), turned to 180 degrees
- moved IC2 32.3 mm to (102.2, 61.3), turned to 0 degrees
- moved C7 25.4 mm to (71.6, 57.4), turned to 180 degrees
- moved C6 22.9 mm to (100.4, 57.2), turned to 180 degrees
- moved R16 11.0 mm to (71.5, 86.3)
- moved R17 11.0 mm to (71.5, 84.5)
- moved TH1 11.0 mm to (71.5, 88.0)
- moved IC3 6.02 mm to (68.0, 61.3)
- moved C37 4.30 mm to (69.7, 105.9), turned to 90 degrees
- moved C22 3.91 mm to (78.5, 106.6)
- moved U2 2.00 mm to (78.7, 103.6), turned to -90 degrees
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Routing:
- net /MCU/PWM_A_H: track 0.00 -> 87.2 mm, vias 0 -> 2
- net /MCU/PWM_A_L: track 0.00 -> 86.4 mm, vias 0 -> 2
- net /MCU/PWM_C_L: track 0.00 -> 52.7 mm, vias 0 -> 2
- net /OUT2: track 37.1 -> 88.0 mm, vias 1 -> 4
- net /MCU/PWM_B_L: track 0.00 -> 48.6 mm, vias 0 -> 2
- net /MCU/PWM_B_H: track 0.00 -> 46.1 mm, vias 0 -> 2
- net /MCU/PWM_C_H: track 0.00 -> 45.7 mm, vias 0 -> 2
- net /OUT1: track 45.2 -> 87.4 mm, vias 1 -> 2
- net /Current_Sens_1: track 0.00 -> 36.7 mm, vias 0 -> 2
- net /Half-Bridge_2/G_L: track 11.5 -> 45.9 mm
- net /OUT3: track 50.6 -> 83.7 mm
- net /Half-Bridge_1/Vshunt_B: track 13.2 -> 41.7 mm, vias 3 -> 4
- net /Half-Bridge_3/G_H: track 6.36 -> 33.0 mm, vias 0 -> 1
- net /Half-Bridge_2/G_H: track 6.36 -> 30.7 mm
- net /Half-Bridge_1/G_H: track 6.36 -> 30.5 mm, vias 0 -> 1
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
Commit message: PCB End of Routing
Parts:
- C12: moved to B.Cu
- moved R7 80.9 mm to (141.3, 83.4), turned to 0 degrees
- moved C12 79.6 mm to (147.8, 71.8)
- moved R46 79.4 mm to (135.0, 103.3)
- moved C10 79.2 mm to (152.3, 101.5)
- moved C11 79.2 mm to (179.2, 71.7)
- moved C16 79.2 mm to (152.3, 107.5)
- moved C17 79.2 mm to (152.3, 112.8), turned to 0 degrees
- moved C26 79.2 mm to (184.4, 87.7)
- moved C27 79.2 mm to (132.3, 103.1)
- moved C30 79.2 mm to (147.2, 96.3)
- moved C33 79.2 mm to (152.2, 103.0)
- moved C34 79.2 mm to (152.2, 104.6)
- moved C37 79.2 mm to (148.7, 112.5)
- moved C42 79.2 mm to (139.2, 80.7)
- moved C46 79.2 mm to (139.2, 77.6)
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Routing:
- net +12V: track 26.5 -> 150.4 mm, vias 2 -> 4
- net +3.3V: track 176.3 -> 229.8 mm
- net GND: track 0.00 -> 38.4 mm, vias 0 -> 69
- net /OUT2: track 88.0 -> 84.7 mm, vias 4 -> 3
- net Net-(IC3-HB): track 8.13 -> 6.79 mm, vias 1 -> 0
- net /Vshunt_3: track 12.8 -> 13.4 mm
- net Net-(IC5-PB8-BOOT0): track 3.25 -> 2.71 mm

Commit message: End of PCB Routing
Parts:
- added G***: LOGO, BassinaLib_LOGO:Bassinga_12_10_logo, F.Cu at (151.5, 81.0)
Routing:
- net GND: vias 69 -> 68
Other:
- board text added: "+"
- board text added: "CAN"
- board text added: "SWD"
- board text added: "U"
- board text added: "UART"
- board text added: "V"
- board text added: "W"
