File: ESC/ESC.kicad_sch (KiCad schematic)
At the start: 50 parts, among them IC1 UCC27211DR, IC2 UCC27211DR, IC3 UCC27211DR, IC5 TCAN3403DDFRQ1, J1 JST SH 3Pin, J2 JST SH 5Pin, J3 JST PH 4Pin

Commit message: Power Supply Update
Parts:
- removed IC1, IC3: UCC27211DR, BassingaLib_BridgeDRVR:SOIC127P600X175-8N, symbol BassingaLib_BridgeDRVR:UCC27211DR
- removed J1: JST SH 3Pin, BassinaLib_Connectors:JST_BM03B-SRSS-TB_LF__SN_, symbol BassinaLib_Connectors:BM03B-SRSS-TB_LF__SN_
- removed R31: 180k 1%, Resistor_SMD:R_0603_1608Metric, symbol Device:R
- added IC4, IC7: UCC27211DR, BassingaLib_BridgeDRVR:SOIC127P600X175-8N, symbol BassingaLib_BridgeDRVR:UCC27211DR
- added J4: MR30PW-M, Connector_AMASS:AMASS_MR30PW-M_1x03_P3.50mm_Horizontal, symbol Connector_Generic:Conn_01x03
- added J6: JST SH 3Pin, BassinaLib_Connectors:JST_BM03B-SRSS-TB_LF__SN_, symbol BassinaLib_Connectors:BM03B-SRSS-TB_LF__SN_
- added R51: 180k 1%, Resistor_SMD:R_0603_1608Metric, symbol Device:R
- S1: value DS04-254-2-01BK-SMT -> SPST Switch
- renumbered C13 to C1, C29 to C10, C3 to C11, C5 to C12, C7 to C13, C30 to C14, C11 to C15, C10 to C16, C9 to C17, C14 to C2, C35 to C3, C34 to C4, C12 to C5, C18 to C6, C19 to C7, C20 to C8, C28 to C9, D3 to D1, D11 to D2, D10 to D3, D9 to D4, IC5 to IC1, IC2 to IC3, J3 to J1, R36 to R1, R17 to R10, R27 to R11, R26 to R12, R28 to R13, R29 to R14, R30 to R15, R38 to R16, R39 to R17, R34 to R18, R33 to R19, R37 to R2, R32 to R20, R47 to R3, R46 to R4, R45 to R5, R40 to R6, R42 to R7, R35 to R9
Connections:
- net Half-Bridge_1/HS is gone; now on net OUT1: C11.2
- net Half-Bridge_2/HS is gone; now on net OUT2: C12.2, IC3.4 (HS)
- net Half-Bridge_3/HS is gone; now on net OUT3: C13.2
- net +12V: now also IC4.1 (VDD), IC7.1 (VDD)
- net GND: now also IC4.7 (VSS), IC7.7 (VSS), J6.2, J6.S1 (SHIELD), J6.S2 (SHIELD)
- net Half-Bridge_1/G_H: now also IC7.3 (HO)
- net Half-Bridge_1/G_L: now also IC7.8 (LO)
- net Half-Bridge_3/G_H: now also IC4.3 (HO)
- net Half-Bridge_3/G_L: now also IC4.8 (LO)
- net MCU/PWM_A_H: now also IC7.5 (HI)
- net MCU/PWM_A_L: now also IC7.6 (LI)
- net MCU/PWM_C_H: now also IC4.5 (HI)
- net MCU/PWM_C_L: now also IC4.6 (LI)
- net OUT1: now also IC7.4 (HS), J4.1 (Pin_1)
- net OUT2: now also J4.2 (Pin_2)
- net OUT3: now also IC4.4 (HS), J4.3 (Pin_3)
- net Vbus_Mesure: now also R51.1
- net at R4.1: now also J6.1
- net at R5.1: now also J6.3
- net at C13.1: now also IC4.2 (HB)
- net at C11.1: now also IC7.2 (HB)
Other:
- sheet Half-Bridge_1 ports: added none; removed HS
- sheet Half-Bridge_2 ports: added none; removed HS
- sheet Half-Bridge_3 ports: added none; removed HS
- moved on the sheet: R3, S1

Commit message: Update 20.07.2025
Parts:
- renumbered IC7 to IC2, J6 to J3, R51 to R8
Changed lines of the file:
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@@
 		(on_board yes)
 		(dnp no)
-		(property "Reference" "IC7"
+		(property "Reference" "IC2"
 			(at 300.482 176.276 0)
 			(effects
@@
 			(project "ESC"
 				(path "/7036a814-0f41-4c6c-a077-a78d90a22423"
-					(reference "IC7")
+					(reference "IC2")
 					(unit 1)
 				)
@@
 		(on_board yes)
 		(dnp no)
-		(property "Reference" "J6"
+		(property "Reference" "J3"
 			(at 60.96 163.576 0)
 			(effects
@@
 			(project ""
 				(path "/7036a814-0f41-4c6c-a077-a78d90a22423"
-					(reference "J6")
+					(reference "J3")
 					(unit 1)
 				)
@@
 		(on_board yes)
 		(dnp no)
-		(property "Reference" "R51"
+		(property "Reference" "R8"
 			(at 177.292 353.822 90)
 			(effects
@@
 			(project "ESC"
 				(path "/7036a814-0f41-4c6c-a077-a78d90a22423"
-					(reference "R51")
+					(reference "R8")
 					(unit 1)
 				)

Commit message: End of Schematic
Changed lines of the file:
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@@
 		)
 	)
-	(text_box "The voltage ragne from:\n\nOut : 0V to 6S_Power (22.2V0)\nPhase: 0V to 2.76V"
+	(text_box "The voltage ragne from:\n\nOut : 0V to +22V2\nPhase: 0V to 2.76V"
 		(exclude_from_sim no)
 		(at 318.77 374.65 0)
@@
 			)
 		)
-		(property "Value" "6S_Power"
+		(property "Value" "+22V"
 			(at 180.34 343.662 0)
 			(effects

Commit message: Start of PCB Layout
Connections:
- net +22V: now reaches R8.2
Changed lines of the file:
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@@
 		(on_board no)
 		(dnp no)
-		(property "Reference" "#PWR017"
+		(property "Reference" "#PWR17"
 			(at 180.34 341.884 0)
 			(effects
@@
 			(project "NovaDrone"
 				(path "/7036a814-0f41-4c6c-a077-a78d90a22423"
-					(reference "#PWR017")
+					(reference "#PWR17")
 					(unit 1)
 				)

Commit message: PCB nearly completed
Connections:
- net MCU/UART2_RX: now also D1.2; no longer D1.1
- net MCU/UART2_TX: now also D1.1; no longer D1.2
- net OUT1: no longer R11.1, R14.1
- net OUT2: now also R11.1
- net OUT3: now also R14.1
- net Phase_2: now also C10.2, R11.2, R13.2; no longer C14.2, R14.2, R15.2
- net Phase_3: now also C14.2, R14.2, R15.2; no longer C10.2, R11.2, R13.2
Changed lines of the file:
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@@
+	)
+	(junction
+		(at 116.84 158.75)
+		(diameter 0)
+		(color 0 0 0 0)
 	)
 	(junction
@@
 	)
 	(junction
+		(at 124.46 162.56)
+		(diameter 0)
+		(color 0 0 0 0)
+	)
+	(junction
 		(at 435.61 275.59)
 		(diameter 0)
@@
 	(junction
 		(at 435.61 231.14)
-		(diameter 0)
-		(color 0 0 0 0)
-	)
-	(junction
-		(at 116.84 162.56)
-		(diameter 0)
-		(color 0 0 0 0)
-	)
-	(junction
-		(at 124.46 158.75)
 		(diameter 0)
 		(color 0 0 0 0)
@@
 	(wire
 		(pts
+			(xy 116.84 158.75) (xy 116.84 166.37)
+		)
+		(stroke
+			(width 0)
+			(type default)
+		)
+	)
+	(wire
+		(pts
 			(xy 435.61 275.59) (xy 426.72 275.59)
 		)
@@
 	(wire
 		(pts
+			(xy 116.84 158.75) (xy 158.75 158.75)
+		)
+		(stroke
+			(width 0)
+			(type default)
+		)
+	)
+	(wire
+		(pts
 			(xy 91.44 44.45) (xy 104.14 44.45)
 		)
@@
 	(wire
 		(pts
+			(xy 124.46 162.56) (xy 154.94 162.56)
+		)
+		(stroke
+			(width 0)
+			(type default)
+		)
+	)
+	(wire
+		(pts
 			(xy 313.69 185.42) (xy 316.23 185.42)
 		)
@@
 	(wire
 		(pts
-			(xy 116.84 162.56) (xy 154.94 162.56)
+			(xy 102.87 162.56) (xy 124.46 162.56)
 		)
 		(stroke
@@
 	(wire
 		(pts
-			(xy 124.46 158.75) (xy 158.75 158.75)
-		)
-		(stroke
-			(width 0)
-			(type default)
-		)
-	)
-	(wire
-		(pts
 			(xy 69.85 73.66) (xy 104.14 73.66)
 		)
@@
 	(wire
 		(pts
-			(xy 102.87 158.75) (xy 124.46 158.75)
+			(xy 102.87 158.75) (xy 116.84 158.75)
 		)
 		(stroke
@@
 	(wire
 		(pts
-			(xy 124.46 158.75) (xy 124.46 166.37)
-		)
-		(stroke
-			(width 0)
-			(type default)
-		)
-	)
-	(wire
-		(pts
 			(xy 341.63 360.68) (xy 341.63 359.41)
 		)
@@
 	(wire
 		(pts
-			(xy 102.87 162.56) (xy 116.84 162.56)
-		)
-		(stroke
-			(width 0)
-			(type default)
-		)
-	)
-	(wire
-		(pts
 			(xy 420.37 356.87) (xy 420.37 353.06)
 		)
@@
 	(wire
 		(pts
-			(xy 116.84 162.56) (xy 116.84 166.37)
-		)
-		(stroke
-			(width 0)
-			(type default)
-		)
-	)
-	(wire
-		(pts
 			(xy 288.29 347.98) (xy 303.53 347.98)
 		)
@@
 		(pts
 			(xy 330.2 210.82) (xy 330.2 222.25)
+		)
+		(stroke
+			(width 0)
+			(type default)
+		)
+	)
+	(wire
+		(pts
+			(xy 124.46 162.56) (xy 124.46 166.37)
 		)
 		(stroke
@@
 		)
 	)
-	(label "OUT1"
+	(label "OUT2"
 		(at 250.19 374.65 0)
 		(effects
@@
 		)
 	)
-	(label "OUT1"
+	(label "OUT3"
 		(at 316.23 347.98 0)
 		(effects
@@
 		)
 	)
-	(label "Phase_3"
+	(label "Phase_2"
 		(at 303.53 374.65 180)
 		(effects
@@
 		)
 	)
-	(label "Phase_2"
+	(label "Phase_3"
 		(at 369.57 347.98 180)
 		(effects

Commit message: BOM
Parts:
- J4: now left out of the parts list
Changed lines of the file:
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@@
 		(unit 1)
 		(exclude_from_sim no)
-		(in_bom yes)
+		(in_bom no)
 		(on_board yes)
 		(dnp no)

Commit message: BOM Update
Parts:
- J1, J2, J3: now left out of the parts list
- R4, R5: Manufacturer_Part_Number AC0603FR-0722RL -> RT0603FRD0722RL
Changed lines of the file:
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@@
 			)
 		)
-		(property "Datasheet" "https://www.mouser.fr/datasheet/2/447/PYu_AC_51_RoHS_L_11-3418659.pdf"
+		(property "Datasheet" "https://www.mouser.fr/datasheet/2/447/PYu_RT_1_to_0_01_RoHS_L_12-3003070.pdf"
 			(at 99.06 158.75 0)
 			(effects
@@
 			)
 		)
-		(property "Manufacturer_Part_Number" "AC0603FR-0722RL"
+		(property "Manufacturer_Part_Number" "RT0603FRD0722RL"
 			(at 99.06 158.75 0)
 			(effects
@@
 	)
 	(symbol
-		(lib_id "Device:R")
-		(at 99.06 162.56 90)
-		(mirror x)
-		(unit 1)
-		(exclude_from_sim no)
-		(in_bom yes)
-		(on_board yes)
-		(dnp no)
-		(property "Reference" "R5"
-			(at 105.156 165.608 90)
-			(effects
-				(font
-					(size 1.27 1.27)
-				)
-				(justify left)
-			)
-		)
-		(property "Value" "22R 1%"
-			(at 99.568 165.608 90)
-			(effects
-				(font
-					(size 1.27 1.27)
-				)
-				(justify left)
-			)
-		)
-		(property "Footprint" "Resistor_SMD:R_0603_1608Metric"
-			(at 99.06 160.782 90)
-			(effects
-				(font
-					(size 1.27 1.27)
-				)
-				(hide yes)
-			)
-		)
-		(property "Datasheet" "https://www.mouser.fr/datasheet/2/447/PYu_AC_51_RoHS_L_11-3418659.pdf"
-			(at 99.06 162.56 0)
-			(effects
-				(font
-					(size 1.27 1.27)
-				)
-				(hide yes)
-			)
-		)
-		(property "Description" "Thick Film Resistors - SMD 22 Ohms 100m W 0603 1% AEC-Q200 Standard"
-			(at 99.06 162.56 0)
-			(effects
-				(font
-					(size 1.27 1.27)
-				)
-				(hide yes)
-			)
-		)
-		(property "Manufacturer_Name" "YAGEO"
-			(at 99.06 162.56 0)
-			(effects
-				(font
-					(size 1.27 1.27)
-				)
-				(hide yes)
-			)
-		)
-		(property "Manufacturer_Part_Number" "AC0603FR-0722RL"
-			(at 99.06 162.56 0)
-			(effects
-				(font
-					(size 1.27 1.27)
-				)
-				(hide yes)
-			)
-		)
-		(property "Packaging" "0603 (608mm)"
-			(at 99.06 162.56 0)
-			(effects
-				(font
-					(size 1.27 1.27)
-				)
-				(hide yes)
-			)
-		)
-		(pin "1"
-		)
-		(pin "2"
-		)
-		(instances
-			(project "NovaDrone"
-				(path "/7036a814-0f41-4c6c-a077-a78d90a22423"
-					(reference "R5")
-					(unit 1)
-				)
-			)
-		)
-	)
-	(symbol
 		(lib_id "Device:C")
 		(at 279.4 163.83 90)
@@
 		(unit 1)
 		(exclude_from_sim no)
-		(in_bom yes)
+		(in_bom no)
 		(on_board yes)
 		(dnp no)
@@
 		(unit 1)
 		(exclude_from_sim no)
-		(in_bom yes)
+		(in_bom no)
 		(on_board yes)
 		(dnp no)
@@
 	(symbol
 		(lib_id "Device:R")
+		(at 99.06 162.56 90)
+		(mirror x)
+		(unit 1)
+		(exclude_from_sim no)
+		(in_bom yes)
+		(on_board yes)
+		(dnp no)
+		(property "Reference" "R5"
+			(at 105.156 165.608 90)
+			(effects
+				(font
+					(size 1.27 1.27)
+				)
+				(justify left)
+			)
+		)
+		(property "Value" "22R 1%"
+			(at 99.568 165.608 90)
+			(effects
+				(font
+					(size 1.27 1.27)
+				)
+				(justify left)
+			)
+		)
+		(property "Footprint" "Resistor_SMD:R_0603_1608Metric"
+			(at 99.06 160.782 90)
+			(effects
+				(font
+					(size 1.27 1.27)
+				)
+				(hide yes)
+			)
+		)
+		(property "Datasheet" "https://www.mouser.fr/datasheet/2/447/PYu_RT_1_to_0_01_RoHS_L_12-3003070.pdf"
+			(at 99.06 162.56 0)
+			(effects
+				(font
+					(size 1.27 1.27)
+				)
+				(hide yes)
+			)
+		)
+		(property "Description" "Thick Film Resistors - SMD 22 Ohms 100m W 0603 1% AEC-Q200 Standard"
+			(at 99.06 162.56 0)
+			(effects
+				(font
+					(size 1.27 1.27)
+				)
+				(hide yes)
+			)
+		)
+		(property "Manufacturer_Name" "YAGEO"
+			(at 99.06 162.56 0)
+			(effects
+				(font
+					(size 1.27 1.27)
+				)
+				(hide yes)
+			)
+		)
+		(property "Manufacturer_Part_Number" "RT0603FRD0722RL"
+			(at 99.06 162.56 0)
+			(effects
+				(font
+					(size 1.27 1.27)
+				)
+				(hide yes)
+			)
+		)
+		(property "Packaging" "0603 (608mm)"
+			(at 99.06 162.56 0)
+			(effects
+				(font
+					(size 1.27 1.27)
+				)
+				(hide yes)
+			)
+		)
+		(pin "1"
+		)
+		(pin "2"
+		)
+		(instances
+			(project "ESC"
+				(path "/7036a814-0f41-4c6c-a077-a78d90a22423"
+					(reference "R5")
+					(unit 1)
+				)
+			)
+		)
+	)
+	(symbol
+		(lib_id "Device:R")
 		(at 107.95 370.84 0)
 		(mirror y)
@@
 		(unit 1)
 		(exclude_from_sim no)
-		(in_bom yes)
+		(in_bom no)
 		(on_board yes)
 		(dnp no)

Commit message: Components library added
Parts:
- J1, J2, J3, J4: now in the parts list
- R4: Manufacturer_Part_Number RT0603FRD0722RL -> AC0603FR-0722RL
Changed lines of the file:
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@@
 			)
 		)
-		(property "Datasheet" "https://www.mouser.fr/datasheet/2/447/PYu_RT_1_to_0_01_RoHS_L_12-3003070.pdf"
+		(property "Datasheet" "https://www.mouser.fr/datasheet/2/447/PYu_AC_51_RoHS_L_11-3418659.pdf"
 			(at 99.06 158.75 0)
 			(effects
@@
 			)
 		)
-		(property "Manufacturer_Part_Number" "RT0603FRD0722RL"
+		(property "Manufacturer_Part_Number" "AC0603FR-0722RL"
 			(at 99.06 158.75 0)
 			(effects
@@
 		(unit 1)
 		(exclude_from_sim no)
-		(in_bom no)
+		(in_bom yes)
 		(on_board yes)
 		(dnp no)
@@
 		(unit 1)
 		(exclude_from_sim no)
-		(in_bom no)
+		(in_bom yes)
 		(on_board yes)
 		(dnp no)
@@
 		(unit 1)
 		(exclude_from_sim no)
-		(in_bom no)
+		(in_bom yes)
 		(on_board yes)
 		(dnp no)
@@
 			)
 		)
-		(property "Datasheet" "~"
+		(property "Datasheet" ""
 			(at 552.45 217.17 0)
 			(effects
@@
 		(unit 1)
 		(exclude_from_sim no)
-		(in_bom no)
+		(in_bom yes)
 		(on_board yes)
 		(dnp no)
