File: ESC/ESC.kicad_sch (KiCad schematic)
At the start: 51 parts, among them IC1 TCAN3403DDFRQ1, IC2 UCC27211DR, IC3 UCC27211DR, IC4 UCC27211DR, J1 JST PH 4Pin, J2 JST SH 5Pin, J3 JST SH 3Pin, J4 MR30PW-M

Commit message: Fly controller design started
Other:
- company: BASSINGA -> BASSINGA_LAB
- title: NovaDrone -> ESC
Changed lines of the file:
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@@
 	(paper "A2")
 	(title_block
-		(title "NovaDrone")
+		(title "ESC")
 		(date "2025-05-21")
-		(rev "v1.0")
-		(company "BASSINGA")
+		(rev "v0.0")
+		(company "BASSINGA_LAB")
+		(comment 1 "Copyright © 2025 Andresse Brisel BASSINGA ")
 	)
 	(rectangle
