File: ESC/Half_Bridge.kicad_sch (KiCad schematic)
At the start: 14 parts, among them Q3 SQJA06EP-T1_GE3, Q4 SQJA06EP-T1_GE3, U1 INA181A1IDBVR

Commit message: Power Supply Update
Parts:
- added C20: 15nF, Capacitor_SMD:C_0603_1608Metric, symbol Device:C
- added R28: 1R 1%, Resistor_SMD:R_0603_1608Metric, symbol Device:R
- U1: footprint SOT95P280X145-6N -> BassingaLib_Sensors:SOT95P280X145-6N
- renumbered C21 to C18, C1 to C19, D2 to D5, D1 to D6, Q4 to Q1, Q3 to Q2, R10 to R21, R11 to R22, R12 to R23, R13 to R24, R3 to R25, R2 to R26, R1 to R27
Connections:
- net Power_GND: now also C20.1
- net HS renamed OUT
- net OUT: now also R28.1
- new net: C20.2, R28.2
Other:
- moved on the sheet: C18, C19, D5, D6, Q1, Q2, R21, R22, R23, R24, R25, R26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

Commit message: End of Schematic
Changed lines of the file:
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@@
 			)
 		)
-		(property "Value" "6S_Power"
+		(property "Value" "+22V"
 			(at 104.14 16.51 0)
 			(effects

Commit message: Start of PCB Layout
Connections:
- net +22V: now reaches C18.1, Q1.5
Changed lines of the file:
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@@
 		(on_board no)
 		(dnp no)
-		(property "Reference" "#PWR038"
+		(property "Reference" "#PWR38"
 			(at 104.14 15.494 0)
 			(effects
@@
 			(project "NovaDrone"
 				(path "/7036a814-0f41-4c6c-a077-a78d90a22423/3d63b6fa-9b75-44ef-b487-19f1bfbe12f4"
-					(reference "#PWR054")
+					(reference "#PWR54")
 					(unit 1)
 				)
 				(path "/7036a814-0f41-4c6c-a077-a78d90a22423/60c9f1ab-8310-4b41-87cd-18a1725e670c"
-					(reference "#PWR038")
+					(reference "#PWR38")
 					(unit 1)
 				)
 				(path "/7036a814-0f41-4c6c-a077-a78d90a22423/f138b3a8-ec69-4954-8088-e3c29779a6aa"
-					(reference "#PWR046")
+					(reference "#PWR46")
 					(unit 1)
 				)

Commit message: BOM Update
Parts:
- R27: Manufacturer_Name YAGEO -> Bourns; Manufacturer_Part_Number PA2512FKE7T0R01E -> CRF2512-FZ-R010ELF
Changed lines of the file:
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@@
 			)
 		)
-		(property "Datasheet" "https://www.yageo.com/upload/media/product/app/datasheet/rchip/pyu-pa_e_51_rohs.pdf"
+		(property "Datasheet" "https://www.mouser.fr/datasheet/2/54/crf-937137.pdf"
 			(at 104.14 80.01 0)
 			(effects
@@
 			)
 		)
-		(property "Description" "Current Sense Resistors - SMD 10 mOhms 3 Watts 1 % 50 ppm/C AEC-Q200"
+		(property "Description" "Current Sense Resistors - SMD 0.010 ohms 1% 75PPM"
 			(at 104.14 80.01 0)
 			(effects
@@
 			)
 		)
-		(property "Manufacturer_Name" "YAGEO"
+		(property "Manufacturer_Name" "Bourns"
 			(at 104.14 80.01 0)
 			(effects
@@
 			)
 		)
-		(property "Manufacturer_Part_Number" "PA2512FKE7T0R01E"
+		(property "Manufacturer_Part_Number" "CRF2512-FZ-R010ELF"
 			(at 104.14 80.01 0)
 			(effects

Commit message: Components library added
Parts:
- R27: Manufacturer_Name Bourns -> YAGEO; Manufacturer_Part_Number CRF2512-FZ-R010ELF -> PA2512FKE7T0R01E
Changed lines of the file:
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@@
 			)
 		)
-		(property "Datasheet" "https://www.mouser.fr/datasheet/2/54/crf-937137.pdf"
+		(property "Datasheet" "https://www.yageo.com/upload/media/product/app/datasheet/rchip/pyu-pa_e_51_rohs.pdf"
 			(at 104.14 80.01 0)
 			(effects
@@
 			)
 		)
-		(property "Description" "Current Sense Resistors - SMD 0.010 ohms 1% 75PPM"
+		(property "Description" "Current Sense Resistors - SMD 10 mOhms 3 Watts 1 % 50 ppm/C AEC-Q200"
 			(at 104.14 80.01 0)
 			(effects
@@
 			)
 		)
-		(property "Manufacturer_Name" "Bourns"
+		(property "Manufacturer_Name" "YAGEO"
 			(at 104.14 80.01 0)
 			(effects
@@
 			)
 		)
-		(property "Manufacturer_Part_Number" "CRF2512-FZ-R010ELF"
+		(property "Manufacturer_Part_Number" "PA2512FKE7T0R01E"
 			(at 104.14 80.01 0)
 			(effects

Commit message: Fly controller design started
Other:
- company: BASSINGA -> BASSINGA_LAB
- title: NovaDrone -> ESC
Changed lines of the file:
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@@
 	(paper "A5")
 	(title_block
-		(title "NovaDrone")
+		(title "ESC")
 		(date "2025-05-21")
-		(rev "v1.0")
-		(company "BASSINGA")
+		(rev "v0.0")
+		(company "BASSINGA_LAB")
+		(comment 1 "Copyright © 2025 Andresse Brisel BASSINGA ")
 	)
 	(text_box "The Gain of the Amplifier is 20V/V\n\nThe maximum current that can be sens is 15A\nV_IS	----> Volt\nI		----> Ampere\n\nI = V_IS/(R_sens*20)"
