File: ESC/MCU.kicad_sch (KiCad schematic)
At the start: 17 parts, among them IC4 STM32G473CCT3, Y1 ECS-80-10-30B-CWN-TR

Commit message: Power Supply Update
Parts:
- added C48: 15nF, Capacitor_SMD:C_0603_1608Metric, symbol Device:C
- IC5: renamed from IC4; footprint QFP50P900X900X160-48N -> BassingaLib_MCU:QFP50P900X900X160-48N
- renumbered C17 to C27, C33 to C28, C32 to C29, C31 to C30, C16 to C31, C25 to C32, C24 to C33, C8 to C34, C15 to C35, C27 to C36, C26 to C37, R43 to R45, R41 to R46, R44 to R47
Connections:
- net +3.3V: now also C48.2
- net GND: now also C48.1
Other:
- moved on the sheet: C32, C33, C36, C37

Commit message: Update 20.07.2025
Parts:
- renumbered C37 to C31, C31 to C32, C36 to C33, C48 to C34, C32 to C35, C33 to C36, C34 to C37, C35 to C38
Changed lines of the file:
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@@
 		(on_board yes)
 		(dnp no)
-		(property "Reference" "C48"
+		(property "Reference" "C34"
 			(at 130.81 157.734 90)
 			(effects
@@
 			(project "ESC"
 				(path "/7036a814-0f41-4c6c-a077-a78d90a22423/480a7603-8487-4f1e-a6dc-719e11c8e32d"
-					(reference "C48")
+					(reference "C34")
 					(unit 1)
 				)
@@
 		(on_board yes)
 		(dnp no)
-		(property "Reference" "C31"
+		(property "Reference" "C32"
 			(at 120.396 43.18 90)
 			(effects
@@
 			(project "NovaDrone"
 				(path "/7036a814-0f41-4c6c-a077-a78d90a22423/480a7603-8487-4f1e-a6dc-719e11c8e32d"
-					(reference "C31")
+					(reference "C32")
 					(unit 1)
 				)
@@
 		(dnp no)
 		(fields_autoplaced yes)
-		(property "Reference" "#PWR071"
+		(property "Reference" "#PWR073"
 			(at 146.05 134.62 0)
 			(effects
@@
 			(project "NovaDrone"
 				(path "/7036a814-0f41-4c6c-a077-a78d90a22423/480a7603-8487-4f1e-a6dc-719e11c8e32d"
-					(reference "#PWR071")
+					(reference "#PWR073")
 					(unit 1)
 				)
@@
 		(on_board yes)
 		(dnp no)
-		(property "Reference" "C36"
+		(property "Reference" "C33"
 			(at 127 157.734 90)
 			(effects
@@
 			(project "NovaDrone"
 				(path "/7036a814-0f41-4c6c-a077-a78d90a22423/480a7603-8487-4f1e-a6dc-719e11c8e32d"
-					(reference "C36")
+					(reference "C33")
 					(unit 1)
 				)
@@
 		(dnp no)
 		(fields_autoplaced yes)
-		(property "Reference" "#PWR074"
+		(property "Reference" "#PWR076"
 			(at 176.53 54.61 0)
 			(effects
@@
 			(project "NovaDrone"
 				(path "/7036a814-0f41-4c6c-a077-a78d90a22423/480a7603-8487-4f1e-a6dc-719e11c8e32d"
-					(reference "#PWR074")
+					(reference "#PWR076")
 					(unit 1)
 				)
@@
 			)
 		)
-		(property "Description" "Standard LEDs - SMD 0603 Dome Lens LED Blue- 465nm 2.65V 2mA"
+		(property "Description" "Standard LEDs - SMD 0603 Dome Lens LED Blue- 465nm"
 			(at 192.532 127.508 0)
 			(effects
@@
 		(dnp no)
 		(fields_autoplaced yes)
-		(property "Reference" "#PWR072"
+		(property "Reference" "#PWR074"
 			(at 165.1 152.4 0)
 			(effects
@@
 			(project "NovaDrone"
 				(path "/7036a814-0f41-4c6c-a077-a78d90a22423/480a7603-8487-4f1e-a6dc-719e11c8e32d"
-					(reference "#PWR072")
+					(reference "#PWR074")
 					(unit 1)
 				)
@@
 		(dnp no)
 		(fields_autoplaced yes)
-		(property "Reference" "#PWR070"
+		(property "Reference" "#PWR072"
 			(at 142.24 27.94 0)
 			(effects
@@
 			(project "NovaDrone"
 				(path "/7036a814-0f41-4c6c-a077-a78d90a22423/480a7603-8487-4f1e-a6dc-719e11c8e32d"
-					(reference "#PWR070")
+					(reference "#PWR072")
 					(unit 1)
 				)
@@
 		(dnp no)
 		(fields_autoplaced yes)
-		(property "Reference" "#PWR081"
+		(property "Reference" "#PWR069"
 			(at 110.49 152.4 0)
 			(effects
@@
 			(project "NovaDrone"
 				(path "/7036a814-0f41-4c6c-a077-a78d90a22423/480a7603-8487-4f1e-a6dc-719e11c8e32d"
-					(reference "#PWR081")
+					(reference "#PWR069")
 					(unit 1)
 				)
@@
 		(dnp no)
 		(fields_autoplaced yes)
-		(property "Reference" "#PWR078"
+		(property "Reference" "#PWR080"
 			(at 200.66 64.77 0)
 			(effects
@@
 			(project "NovaDrone"
 				(path "/7036a814-0f41-4c6c-a077-a78d90a22423/480a7603-8487-4f1e-a6dc-719e11c8e32d"
-					(reference "#PWR078")
+					(reference "#PWR080")
 					(unit 1)
 				)
@@
 		(dnp no)
 		(fields_autoplaced yes)
-		(property "Reference" "#PWR076"
+		(property "Reference" "#PWR078"
 			(at 176.53 137.16 0)
 			(effects
@@
 			(project "NovaDrone"
 				(path "/7036a814-0f41-4c6c-a077-a78d90a22423/480a7603-8487-4f1e-a6dc-719e11c8e32d"
-					(reference "#PWR076")
+					(reference "#PWR078")
 					(unit 1)
 				)
@@
 		(dnp no)
 		(fields_autoplaced yes)
-		(property "Reference" "#PWR077"
+		(property "Reference" "#PWR079"
 			(at 199.39 146.05 0)
 			(effects
@@
 			(project "NovaDrone"
 				(path "/7036a814-0f41-4c6c-a077-a78d90a22423/480a7603-8487-4f1e-a6dc-719e11c8e32d"
-					(reference "#PWR077")
+					(reference "#PWR079")
 					(unit 1)
 				)
@@
 		(on_board yes)
 		(dnp no)
-		(property "Reference" "C33"
+		(property "Reference" "C36"
 			(at 161.29 157.734 90)
 			(effects
@@
 			(project "NovaDrone"
 				(path "/7036a814-0f41-4c6c-a077-a78d90a22423/480a7603-8487-4f1e-a6dc-719e11c8e32d"
-					(reference "C33")
+					(reference "C36")
 					(unit 1)
 				)
@@
 		(dnp no)
 		(fields_autoplaced yes)
-		(property "Reference" "#PWR075"
+		(property "Reference" "#PWR077"
 			(at 176.53 118.11 0)
 			(effects
@@
 			(project "NovaDrone"
 				(path "/7036a814-0f41-4c6c-a077-a78d90a22423/480a7603-8487-4f1e-a6dc-719e11c8e32d"
-					(reference "#PWR075")
+					(reference "#PWR077")
 					(unit 1)
 				)
@@
 		(dnp no)
 		(fields_autoplaced yes)
-		(property "Reference" "#PWR080"
+		(property "Reference" "#PWR070"
 			(at 115.57 172.72 0)
 			(effects
@@
 			(project "NovaDrone"
 				(path "/7036a814-0f41-4c6c-a077-a78d90a22423/480a7603-8487-4f1e-a6dc-719e11c8e32d"
-					(reference "#PWR080")
+					(reference "#PWR070")
 					(unit 1)
 				)
@@
 		(on_board yes)
 		(dnp no)
-		(property "Reference" "C34"
+		(property "Reference" "C37"
 			(at 172.72 123.444 90)
 			(effects
@@
 			(project "NovaDrone"
 				(path "/7036a814-0f41-4c6c-a077-a78d90a22423/480a7603-8487-4f1e-a6dc-719e11c8e32d"
-					(reference "C34")
+					(reference "C37")
 					(unit 1)
 				)
@@
 		(on_board yes)
 		(dnp no)
-		(property "Reference" "C35"
+		(property "Reference" "C38"
 			(at 187.706 52.07 90)
 			(effects
@@
 			(project "NovaDrone"
 				(path "/7036a814-0f41-4c6c-a077-a78d90a22423/480a7603-8487-4f1e-a6dc-719e11c8e32d"
-					(reference "C35")
+					(reference "C38")
 					(unit 1)
 				)
@@
 		(dnp no)
 		(fields_autoplaced yes)
-		(property "Reference" "#PWR073"
+		(property "Reference" "#PWR075"
 			(at 165.1 171.45 0)
 			(effects
@@
 			(project "NovaDrone"
 				(path "/7036a814-0f41-4c6c-a077-a78d90a22423/480a7603-8487-4f1e-a6dc-719e11c8e32d"
-					(reference "#PWR073")
+					(reference "#PWR075")
 					(unit 1)
 				)
@@
 		(on_board yes)
 		(dnp no)
-		(property "Reference" "C32"
+		(property "Reference" "C35"
 			(at 148.59 157.734 90)
 			(effects
@@
 			(project "NovaDrone"
 				(path "/7036a814-0f41-4c6c-a077-a78d90a22423/480a7603-8487-4f1e-a6dc-719e11c8e32d"
-					(reference "C32")
+					(reference "C35")
 					(unit 1)
 				)
@@
 		(dnp no)
 		(fields_autoplaced yes)
-		(property "Reference" "#PWR079"
+		(property "Reference" "#PWR081"
 			(at 200.66 82.55 0)
 			(effects
@@
 			(project "NovaDrone"
 				(path "/7036a814-0f41-4c6c-a077-a78d90a22423/480a7603-8487-4f1e-a6dc-719e11c8e32d"
-					(reference "#PWR079")
+					(reference "#PWR081")
 					(unit 1)
 				)
@@
 		(on_board yes)
 		(dnp no)
-		(property "Reference" "C37"
+		(property "Reference" "C31"
 			(at 114.3 157.734 90)
 			(effects
@@
 			(project "NovaDrone"
 				(path "/7036a814-0f41-4c6c-a077-a78d90a22423/480a7603-8487-4f1e-a6dc-719e11c8e32d"
-					(reference "C37")
+					(reference "C31")
 					(unit 1)
 				)
@@
 		(dnp no)
 		(fields_autoplaced yes)
-		(property "Reference" "#PWR069"
+		(property "Reference" "#PWR071"
 			(at 130.81 46.99 0)
 			(effects
@@
 			(project "NovaDrone"
 				(path "/7036a814-0f41-4c6c-a077-a78d90a22423/480a7603-8487-4f1e-a6dc-719e11c8e32d"
-					(reference "#PWR069")
+					(reference "#PWR071")
 					(unit 1)
 				)

Commit message: PCB nearly completed
Connections:
- net Phase_3: now also IC5.26 (PB12); no longer IC5.27 (PB13)
- net V12_Mesure: now also IC5.27 (PB13); no longer IC5.28 (PB14)
- net V3.3_Mesure: now also IC5.28 (PB14); no longer IC5.29 (PB15)
- net Vbus_Mesure: now also IC5.29 (PB15); no longer IC5.26 (PB12)
- net at R47.1: now also IC5.33 (PA11); no longer IC5.25 (PB11)
Changed lines of the file:
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@@
 	)
 	(no_connect
+		(at 173.99 100.33)
+	)
+	(no_connect
 		(at 114.3 72.39)
 	)
@@
 		(at 143.51 114.3)
 	)
-	(no_connect
-		(at 173.99 80.01)
-	)
-	(wire
-		(pts
-			(xy 199.39 100.33) (xy 199.39 107.95)
-		)
-		(stroke
-			(width 0)
-			(type default)
-		)
-	)
 	(wire
 		(pts
@@
 	(wire
 		(pts
-			(xy 173.99 74.93) (xy 200.66 74.93)
+			(xy 173.99 74.93) (xy 207.01 74.93)
 		)
 		(stroke
@@
 	(wire
 		(pts
-			(xy 199.39 134.62) (xy 199.39 139.7)
+			(xy 199.39 134.62) (xy 199.39 137.16)
 		)
 		(stroke
@@
 	(wire
 		(pts
+			(xy 199.39 80.01) (xy 173.99 80.01)
+		)
+		(stroke
+			(width 0)
+			(type default)
+		)
+	)
+	(wire
+		(pts
 			(xy 24.13 137.16) (xy 38.1 137.16)
 		)
@@
 	(wire
 		(pts
-			(xy 173.99 100.33) (xy 199.39 100.33)
-		)
-		(stroke
-			(width 0)
-			(type default)
-		)
-	)
-	(wire
-		(pts
 			(xy 124.46 46.99) (xy 130.81 46.99)
 		)
@@
 	(wire
 		(pts
-			(xy 200.66 76.2) (xy 200.66 74.93)
+			(xy 199.39 80.01) (xy 199.39 107.95)
+		)
+		(stroke
+			(width 0)
+			(type default)
+		)
+	)
+	(wire
+		(pts
+			(xy 207.01 77.47) (xy 207.01 74.93)
 		)
 		(stroke
@@
 	(hierarchical_label "Vbus_Mesure"
 		(shape input)
-		(at 180.34 97.79 0)
+		(at 180.34 90.17 0)
 		(effects
 			(font
@@
 	(hierarchical_label "Phase_3"
 		(shape input)
-		(at 180.34 95.25 0)
+		(at 180.34 97.79 0)
 		(effects
 			(font
@@
 	(hierarchical_label "V12_Mesure"
 		(shape input)
-		(at 180.34 92.71 0)
+		(at 180.34 95.25 0)
 		(effects
 			(font
@@
 	(hierarchical_label "V3.3_Mesure"
 		(shape input)
-		(at 180.34 90.17 0)
+		(at 180.34 92.71 0)
 		(effects
 			(font
@@
 	(symbol
 		(lib_id "power:GND")
-		(at 199.39 139.7 0)
+		(at 199.39 137.16 0)
 		(unit 1)
 		(exclude_from_sim no)
@@
 		(fields_autoplaced yes)
 		(property "Reference" "#PWR079"
-			(at 199.39 146.05 0)
+			(at 199.39 143.51 0)
 			(effects
 				(font
@@
 		)
 		(property "Value" "GND"
-			(at 199.39 144.78 0)
+			(at 199.39 142.24 0)
 			(effects
 				(font
@@
 		)
 		(property "Footprint" ""
-			(at 199.39 139.7 0)
+			(at 199.39 137.16 0)
 			(effects
 				(font
@@
 		)
 		(property "Datasheet" ""
-			(at 199.39 139.7 0)
+			(at 199.39 137.16 0)
 			(effects
 				(font
@@
 		)
 		(property "Description" "Power symbol creates a global label with name \"GND\" , ground"
-			(at 199.39 139.7 0)
+			(at 199.39 137.16 0)
 			(effects
 				(font
@@
 	(symbol
 		(lib_id "power:GND")
-		(at 200.66 76.2 0)
+		(at 207.01 77.47 0)
 		(unit 1)
 		(exclude_from_sim no)
@@
 		(fields_autoplaced yes)
 		(property "Reference" "#PWR081"
-			(at 200.66 82.55 0)
+			(at 207.01 83.82 0)
 			(effects
 				(font
@@
 		)
 		(property "Value" "GND"
-			(at 200.66 81.28 0)
+			(at 207.01 82.55 0)
 			(effects
 				(font
@@
 		)
 		(property "Footprint" ""
-			(at 200.66 76.2 0)
+			(at 207.01 77.47 0)
 			(effects
 				(font
@@
 		)
 		(property "Datasheet" ""
-			(at 200.66 76.2 0)
+			(at 207.01 77.47 0)
 			(effects
 				(font
@@
 		)
 		(property "Description" "Power symbol creates a global label with name \"GND\" , ground"
-			(at 200.66 76.2 0)
+			(at 207.01 77.47 0)
 			(effects
 				(font

Commit message: Fly controller design started
Other:
- company: (none) -> BASSINGA_LAB
- title: (none) -> ESC
Changed lines of the file:
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@@
 	(generator_version "9.0")
 	(paper "A4")
+	(title_block
+		(title "ESC")
+		(date "2025-05-21")
+		(rev "v0.0")
+		(company "BASSINGA_LAB")
+		(comment 1 "Copyright © 2025 Andresse Brisel BASSINGA ")
+	)
 	(junction
 		(at 63.5 137.16)
