File: ESC/Power_Supply.kicad_sch (KiCad schematic)
At the start: 23 parts, among them IC6 BD433M5FP-CE2, J5 XT30PW-M

Commit message: Components library added
Parts:
- J5: now in the parts list
Changed lines of the file:
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@@
 		(unit 1)
 		(exclude_from_sim no)
-		(in_bom no)
+		(in_bom yes)
 		(on_board yes)
 		(dnp no)

Commit message: Fly controller design started
Other:
- company: (none) -> BASSINGA_LAB
- title: (none) -> ESC
Changed lines of the file:
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@@
 	(generator_version "9.0")
 	(paper "A4")
+	(title_block
+		(title "ESC")
+		(date "2025-05-21")
+		(rev "v0.0")
+		(company "BASSINGA_LAB")
+		(comment 1 "Copyright © 2025 Andresse Brisel BASSINGA ")
+	)
 	(junction
 		(at 168.91 99.06)
