File: PCU/logic_power_supply.kicad_sch (KiCad schematic)
At the start: 3 parts, among them IC30 BD433M5FP-CE2

Commit message: Logic PSU Completed
Parts:
- removed IC30: BD433M5FP-CE2, BassingaLib_LDO:BD433M5FPCE2, symbol BassingaLib_LDO:BD433M5FP-CE2
- added C193, C220: 15nF, Capacitor_SMD:C_0603_1608Metric, symbol Device:C
- added C225, C231, C237: 10uF 63V, Capacitor_SMD:C_1210_3225Metric, symbol Device:C
- added C226, C230, C233, C234: 0.1uF 50V, Capacitor_SMD:C_0603_1608Metric, symbol Device:C
- added C227: 56pF 50V, Capacitor_SMD:C_0603_1608Metric, symbol Device:C
- added C228, C229, C232, C235, C236, C238, C239: 22uF 25V, Capacitor_SMD:C_1210_3225Metric, symbol Device:C
- added D49, D52: SS0540_R1_00001, BassingaLib_Diodes:SOD3816X135N, symbol BassingaLib_Diodes:SS0540_R1_00001
- added FB2: FerriteBead, Inductor_SMD:L_0805_2012Metric, symbol Device:FerriteBead
- added IC35: AP63205WU-7, BassingaLib_SMPS:AP63205WU7, symbol BassingaLib_SMPS:AP63205WU-7
- added IC36: AP63203WU-7, BassingaLib_SMPS:AP63203WU7, symbol BassingaLib_SMPS:AP63203WU-7
- added J16, J17, J18: B2B-PH-K-S, BassinaLib_Connectors:JST_B2B-PH-K-S, symbol BassinaLib_Connectors:B2B-PH-K-S
- added L3: 10uH 2.2A 20%, BassingaLib_Inductors:BWVS00505040100M00, symbol BassingaLib_Inductors:BWVS00505040100M00
- added L4: 4.7uH 2.9A 20%, BassingaLib_Inductors:ASPI-4030S, symbol BassingaLib_Inductors:ASPI-4030S-4R7M-T
- added L6: 3.9uH 3A, 20%, BassingaLib_Inductors:ASPI0628150MT1, symbol BassingaLib_Inductors:ASPI-0628-3R9M-T1
- added LED17: RED LED, BassinaLib_LEDs:LEDM168X80N, symbol BassinaLib_LEDs:APHD1608LSURCK
- added LED18, LED19, LED20: GREEN, BassinaLib_LEDs:LEDM168X80N, symbol BassinaLib_LEDs:APHD1608LZGCK
- added PS3: AP63200WU-7, BassingaLib_SMPS:SOT95P280X100-6N, symbol BassingaLib_SMPS:AP63200WU-7
- added R241, R255, R268, R271: 18k 1%, Resistor_SMD:R_0603_1608Metric, symbol Device:R
- added R242: 2k 1%, Resistor_SMD:R_0603_1608Metric, symbol Device:R
- added R254: 180k 1%, Resistor_SMD:R_0603_1608Metric, symbol Device:R
- added R267: 249k 1%, Resistor_SMD:R_0603_1608Metric, symbol Device:R
- added R269: 0.22R 1%, Resistor_SMD:R_0805_2012Metric, symbol Device:R
- added R270: 6.8k 1%, Resistor_SMD:R_0603_1608Metric, symbol Device:R
- added R272: 100k 1%, Resistor_SMD:R_0603_1608Metric, symbol Device:R
- added R273, R274: 68k 1%, Resistor_SMD:R_0603_1608Metric, symbol Device:R
- added R275: 10k 1%, Resistor_SMD:R_0603_1608Metric, symbol Device:R
- added R276, R277: 33k 1%, Resistor_SMD:R_0603_1608Metric, symbol Device:R
- added TP10, TP11, TP9: TestPoint, TestPoint:TestPoint_Pad_D1.0mm, symbol Connector:TestPoint
- added TP8: TestPoint, symbol Connector:TestPoint
- C141: value 4.7uF 50V -> 15nF; footprint Capacitor_SMD:C_1206_3216Metric -> Capacitor_SMD:C_0603_1608Metric; Manufacturer_Part_Number CL31B475KBHNFNE -> CL10B153KB8NNNC; Packaging 1206 (3216 mm) -> 0603 (608mm)
- C145: value 10uF 63V -> 15nF; footprint Capacitor_SMD:C_1210_3225Metric -> Capacitor_SMD:C_0603_1608Metric; Manufacturer_Part_Number CL32B106KMVNNWE -> CL10B153KB8NNNC; Packaging 1210 (3225mm) -> 0603 (608mm)
Connections:
- net +12V_ is gone; now on net GND: C141.1
- net +3.3V_Logic: now also C232.2, C233.2, D49.1 (K), D52.1 (K), J18.1 (P), R242.1, R269.1, R276.2, TP9.1; no longer C145.2
- net +Vbat: now also C225.2, C231.2, C237.2, IC35.2 (EN), IC35.3 (VIN), IC36.2 (EN), IC36.3 (VIN), PS3.2 (EN), PS3.3 (VIN), R241.1, R254.2
- net GND: now also C193.1, C220.1, C225.1, C228.1, C229.1, C231.1, C232.1, C233.1, C235.1, C236.1, C237.1, C238.1, C239.1, IC35.4 (GND), IC36.4 (GND), J16.N (2), J17.N (2), J18.N (2), LED17.1 (K), LED18.1 (K), LED19.1 (K), LED20.1 (K), PS3.4 (GND), R255.1, R268.1, R273.1, R275.2, R277.1; no longer C141.2
- new net: C227.1, PS3.1 (FB), R267.1, R268.2
- new net: C226.2, PS3.6 (BST)
- new net: LED17.2 (A), R241.2
- new net: LED20.2 (A), R271.2
- new net: C230.1, IC36.5 (SW), L6.1
- new net: C235.2, C236.2, FB2.1, IC36.1 (FB), L6.2, TP10.1
- new net: C230.2, IC36.6 (BST)
- new net: FB2.2, R269.2
- new net: LED18.2 (A), R242.2
- new net: LED19.2 (A), R270.2
- new net: C234.1, IC35.5 (SW), L4.1
- new net: C234.2, IC35.6 (BST)
- new net +12V_Logic: C227.2, C228.2, C229.2, J16.1 (P), L3.2, R267.2, R271.1, R274.2, TP8.1
- new net +5V_Logic: C238.2, C239.2, IC35.1 (FB), J17.1 (P), L4.2, R270.1, R272.2, TP11.1
- new net SW: C226.1, L3.1, PS3.5 (SW)
- new net V12Logic_Mesure: C145.2, D52.2 (A), R274.1, R275.1
- new net V3.3Logic_Mesure: C193.2, R276.1, R277.2
- new net V5Logic_Mesure: C141.2, R272.1, R273.2
- new net Vbat_Mesure: C220.2, D49.2 (A), R254.1, R255.2
Other:
- note added: "+12V_Logic Mesurement"
- note added: "+3.3V_Logic Mesurement"
- note added: "+5V_Logic Mesurement"
- note added: "12V Logic, 2A Max"
- note added: "3.3V Logic, 2A Max"
- note added: "5V Logic, 2A Max"
- note added: "Battery Voltage Mesurement"
- note added: "Connectors"

Commit message: Supervisor Block
Parts:
- TP10: renamed from TP8; footprint (none) -> TestPoint:TestPoint_Pad_D1.0mm
- renumbered C220 to C205, C225 to C207, C231 to C208, C237 to C209, C145 to C212, C234 to C213, C226 to C214, C230 to C215, C227 to C217, C238 to C218, C235 to C219, C239 to C221, C236 to C222, C141 to C225, C228 to C226, C229 to C227, C232 to C229, C233 to C230, C193 to C231, D49 to D47, D52 to D48, IC35 to IC34, IC36 to IC35, L4 to L3, L3 to L4, L6 to L5, LED20 to LED18, LED18 to LED20, PS3 to PS2, R254 to R237, R255 to R238, R274 to R248, R275 to R249, R272 to R252, R273 to R253, R267 to R255, R268 to R256, R269 to R258, R276 to R259, R277 to R260, R241 to R261, R271 to R262, R270 to R263, R242 to R264, TP9 to TP11, TP11 to TP8, TP10 to TP9
