File: PCU/PCU.kicad_pcb (KiCad board)
At the start: 4 copper layers, 140 x 140 mm, 760 parts, among them IC1 TCAN3403DDFRQ1, IC10 LM321LVIDBVR, IC11 LM321LVIDBVR, IC12 STM32G473CCT3, IC13 TCAN3403DDFRQ1, IC14 UCC27211DR, IC15 UCC27211DR, IC16 UCC27211DR, IC17 LM321LVIDBVR, IC18 LM321LVIDBVR, IC19 LM321LVIDBVR, IC2 UCC27211DR, IC20 STM32G473CCT3, IC21 TCAN3403DDFRQ1, IC22 UCC27211DR, IC23 UCC27211DR, IC24 UCC27211DR, IC25 LM321LVIDBVR, IC26 LM321LVIDBVR, IC27 LM321LVIDBVR, IC28 STM32G473CCT3, IC29 AP63203WU-7, IC3 UCC27211DR, IC30 STM32G473CCT3, IC31 LM321LVIDBVR, IC32 LM5060MMX_NOPB, IC33 LM321LVIDBVR, IC34 AP63205WU-7, IC35 AP63203WU-7, IC36 TCAN3403DDFRQ1, IC37 LM321LVIDBVR, IC38 STM32G473CCT3, IC4 UCC27211DR, IC5 TCAN3403DDFRQ1, IC6 UCC27211DR, IC7 UCC27211DR, IC8 UCC27211DR, IC9 LM321LVIDBVR, J1 XT60PW-M, J10 JST SH 5Pin, J11 JST SH 3Pin, J12 JST SH 5Pin, J13 JST SH 3Pin, J14 JST SH 5Pin, J15 JST SH 3Pin, J16 B2B-PH-K-S, J17 B2B-PH-K-S, J18 B2B-PH-K-S, J19 JST SH 5Pin, J2 B4B-PH-K-S_LF__SN_, J20 JST SH 3Pin, J21 USB4120-03-C, J3 B4B-PH-K-S_LF__SN_, J4 Conn_01x03_Pin, J5 Conn_01x03_Pin, J6 Conn_01x03_Pin, J7 Conn_01x03_Pin, J8 JST SH 5Pin, J9 JST SH 3Pin, Q1 SQJA06EP-T1_GE3, Q10 SQJA06EP-T1_GE3, Q11 SQJA06EP-T1_GE3, Q12 SQJA06EP-T1_GE3, Q13 SQJA06EP-T1_GE3, Q14 SQJA06EP-T1_GE3, Q15 SQJA06EP-T1_GE3, Q16 SQJA06EP-T1_GE3, Q17 SQJA06EP-T1_GE3, Q18 SQJA06EP-T1_GE3, Q19 SQJA06EP-T1_GE3, Q2 SQJA06EP-T1_GE3, Q20 SQJA06EP-T1_GE3, Q21 BC846B, Q22 DMP6023LFG-7, Q23 NTMFS5H600NLT1G, Q24 NTMFS5H600NLT1G, Q25 NTMFS5H600NLT1G, Q26 NTMFS5H600NLT1G, Q27 BC846B, Q28 SQJA06EP-T1_GE3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

Commit message: Power stage routed
Parts:
- moved C240 124.3 mm to (80.0, 119.8), turned to 0 degrees
- moved C197 117.0 mm to (80.0, 117.6), turned to 0 degrees
- moved J4 114.8 mm to (71.8, 101.0), turned to -90 degrees
- moved J5 113.1 mm to (203.2, 79.6), turned to 90 degrees
- moved C211 110.6 mm to (80.0, 93.2), turned to 0 degrees
- moved D46 106.5 mm to (76.4, 112.6), turned to -90 degrees
- moved D13 106.1 mm to (198.6, 68.0), turned to 90 degrees
- moved C43 105.8 mm to (194.4, 63.2), turned to 180 degrees
- moved D43 104.8 mm to (76.4, 98.1), turned to -90 degrees
- moved D15 104.3 mm to (198.6, 82.5), turned to 90 degrees
- moved Q28 103.8 mm to (77.9, 112.7), turned to 90 degrees
- moved Q1 103.4 mm to (197.1, 67.9), turned to -90 degrees
- moved C27 102.6 mm to (195.2, 87.4), turned to 180 degrees
- moved R243 102.4 mm to (78.9, 113.6), turned to 90 degrees
- moved R32 102.0 mm to (196.1, 67.0), turned to -90 degrees
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Routing:
- net /ESC_4/OUT1: track 1.52 -> 22.1 mm, vias 1 -> 4
- net /ESC_1/OUT1: track 1.52 -> 21.9 mm, vias 1 -> 4
- net /ESC_2/OUT1: track 1.52 -> 21.8 mm, vias 1 -> 4
- net /ESC_3/OUT1: track 1.52 -> 21.7 mm, vias 1 -> 4
- net /ESC_3/OUT2: track 1.53 -> 21.3 mm, vias 1 -> 4
- net /ESC_4/OUT2: track 1.53 -> 21.1 mm, vias 1 -> 4
- net /ESC_2/OUT2: track 1.53 -> 21.0 mm, vias 1 -> 4
- net /ESC_1/OUT2: track 1.53 -> 20.8 mm, vias 1 -> 4
- net +Vbus: vias 30 -> 125
- added copper zone on B.Cu, net +Vbus

Commit message: Drivers routed
Parts:
- C10, C11, C114, C115, C116, C117, C118, C119, C18, C19, C20, C21, C22, C23, C6, C67, C68, C7, C70, C71, C8, C9, D2, D3, IC14, IC15, IC16, IC2, IC22, IC23, IC24, IC3, IC4, IC6, IC7, IC8, R1: moved to B.Cu
- moved C109 316.0 mm to (345.2, 162.1)
- moved C110 316.0 mm to (357.5, 162.4)
- moved C111 316.0 mm to (345.2, 164.7)
- moved C112 316.0 mm to (357.5, 165.4)
- moved C113 316.0 mm to (345.2, 167.2)
- moved C120 316.0 mm to (345.2, 177.2)
- moved C133 316.0 mm to (338.1, 174.4)
- moved C141 316.0 mm to (338.0, 170.1)
- moved C144 316.0 mm to (338.3, 188.6)
- moved C146 316.0 mm to (324.7, 184.3)
- moved C147 316.0 mm to (327.7, 184.3)
- moved C148 316.0 mm to (331.7, 186.8)
- moved D28 316.0 mm to (346.3, 180.6)
- moved D29 316.0 mm to (344.4, 174.3)
- moved D30 316.0 mm to (346.3, 185.0)
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Routing:
- net /ESC_4/Half-Bridge_2/G_H: track 2.69 -> 30.1 mm, vias 0 -> 2
- net /ESC_2/Half-Bridge_2/G_H: track 2.69 -> 28.8 mm, vias 0 -> 2
- net /ESC_1/Half-Bridge_2/G_H: track 2.69 -> 27.3 mm
- net /ESC_3/Half-Bridge_2/G_H: track 2.69 -> 25.3 mm
- net +12V_PWR: track 10.9 -> 32.6 mm, vias 3 -> 4
- net /ESC_3/Half-Bridge_1/G_H: track 2.50 -> 23.9 mm, vias 0 -> 2
- net /ESC_4/Half-Bridge_1/G_H: track 2.50 -> 23.5 mm
- net /ESC_1/Half-Bridge_1/G_H: track 2.50 -> 23.3 mm, vias 0 -> 2
- net /ESC_2/Half-Bridge_1/G_H: track 2.50 -> 22.9 mm
- net /ESC_1/OUT1: track 21.9 -> 42.3 mm
- net /ESC_2/OUT2: track 21.0 -> 39.9 mm, vias 4 -> 5
- net /ESC_3/OUT2: track 21.3 -> 40.0 mm, vias 4 -> 5
- net /ESC_1/OUT2: track 20.8 -> 39.4 mm
- net /ESC_4/OUT2: track 21.1 -> 39.4 mm, vias 4 -> 5
- net /ESC_1/Half-Bridge_2/G_L: track 3.22 -> 20.4 mm, vias 0 -> 2
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