File: PCU/PCU.kicad_pcb (KiCad board)
At the start: 4 copper layers, 140 x 140 mm, 755 parts, among them IC1 TCAN3403DDFRQ1, IC10 LM321LVIDBVR, IC11 LM321LVIDBVR, IC12 STM32G473CCT3, IC13 TCAN3403DDFRQ1, IC14 UCC27211DR, IC15 UCC27211DR, IC16 UCC27211DR, IC17 LM321LVIDBVR, IC18 LM321LVIDBVR, IC19 LM321LVIDBVR, IC2 UCC27211DR, IC20 STM32G473CCT3, IC21 TCAN3403DDFRQ1, IC22 UCC27211DR, IC23 UCC27211DR, IC24 UCC27211DR, IC25 LM321LVIDBVR, IC26 LM321LVIDBVR, IC27 LM321LVIDBVR, IC28 STM32G473CCT3, IC29 AP63203WU-7, IC3 UCC27211DR, IC30 STM32G473CCT3, IC31 LM321LVIDBVR, IC32 LM5060MMX_NOPB, IC33 LM321LVIDBVR, IC34 AP63205WU-7, IC35 AP63203WU-7, IC36 TCAN3403DDFRQ1, IC37 LM321LVIDBVR, IC38 STM32G473CCT3, IC4 UCC27211DR, IC5 TCAN3403DDFRQ1, IC6 UCC27211DR, IC7 UCC27211DR, IC8 UCC27211DR, IC9 LM321LVIDBVR, J1 XT60PW-M, J10 JST SH 5Pin, J11 JST SH 3Pin, J12 JST SH 5Pin, J13 JST SH 3Pin, J14 JST SH 5Pin, J15 JST SH 3Pin, J16 B2B-PH-K-S, J17 B2B-PH-K-S, J18 B2B-PH-K-S, J19 JST SH 5Pin, J2 B4B-PH-K-S_LF__SN_, J20 JST SH 3Pin, J21 USB4120-03-C, J3 B4B-PH-K-S_LF__SN_, J4 Conn_01x03_Pin, J5 Conn_01x03_Pin, J6 Conn_01x03_Pin, J7 Conn_01x03_Pin, J8 JST SH 5Pin, J9 JST SH 3Pin, Q1 SQJA06EP-T1_GE3, Q10 SQJA06EP-T1_GE3, Q11 SQJA06EP-T1_GE3, Q12 SQJA06EP-T1_GE3, Q13 SQJA06EP-T1_GE3, Q14 SQJA06EP-T1_GE3, Q15 SQJA06EP-T1_GE3, Q16 SQJA06EP-T1_GE3, Q17 SQJA06EP-T1_GE3, Q18 SQJA06EP-T1_GE3, Q19 SQJA06EP-T1_GE3, Q2 SQJA06EP-T1_GE3, Q20 SQJA06EP-T1_GE3, Q21 BC846B, Q22 DMP6023LFG-7, Q23 NTMFS5H600NLT1G, Q24 NTMFS5H600NLT1G, Q25 NTMFS5H600NLT1G, Q26 NTMFS5H600NLT1G, Q27 BC846B, Q28 SQJA06EP-T1_GE3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

Commit message: Logic power supply routed
Parts:
- moved C3 1.12 mm to (124.3, 102.8), turned to -90 degrees
- moved R196 0.09 mm to (137.5, 61.4)
Routing:
- net +3.3V_Logic_filtered: track 34.0 -> 368.9 mm, vias 8 -> 15
- net +12V_PWR: track 34.6 -> 228.8 mm, vias 3 -> 23
- net +Vbus: track 16.2 -> 61.6 mm
- net /+Vbat: track 74.1 -> 110.7 mm, vias 40 -> 44
- net +12V_Logic: track 10.2 -> 41.9 mm
- net +5V_Logic: track 12.5 -> 30.9 mm, vias 2 -> 3
- net +3.3V_Logic: track 12.4 -> 27.4 mm, vias 2 -> 3
- net Net-(Q22-G): track 16.5 -> 26.9 mm
- net /ESC_2/Half-Bridge_2/G_H: track 33.3 -> 26.3 mm
- net /ESC_4/Half-Bridge_2/G_H: track 33.3 -> 26.3 mm
- net Net-(LED11-A): track 0.00 -> 6.31 mm
- net /Supervisor/nRST: track 129.5 -> 123.4 mm
- net Net-(LED12-A): track 0.00 -> 6.11 mm
- net /Supervisor/push_button: track 83.8 -> 79.5 mm
- net /ESC_3/OUT1: track 56.3 -> 59.7 mm
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- added copper zone on In2.Cu, net /+Vbat
