File: PCU/high_power_supply.kicad_sch (KiCad schematic)
At the start: 54 parts

Commit message: Logic PSU Completed
Parts:
- removed C193: 22uF 25V, Capacitor_SMD:C_1210_3225Metric, symbol Device:C
- removed L2: 6.8uH 2.1A 20%, BassingaLib_Inductors:SDCL1V40206R8MR, symbol BassingaLib_Inductors:SDCL1V4020-6R8M-R
- removed PS2: AP63200WU-7, BassingaLib_SMPS:SOT95P280X100-6N, symbol BassingaLib_SMPS:AP63200WU-7
- removed R241: 196k 1%, Resistor_SMD:R_0603_1608Metric, symbol Device:R
- removed R242: 62k 1%, Resistor_SMD:R_0603_1608Metric, symbol Device:R
- added IC37: AP63203WU-7, BassingaLib_SMPS:AP63203WU7, symbol BassingaLib_SMPS:AP63203WU-7
- added L2: 3.9uH 3A, 20%, BassingaLib_Inductors:ASPI0628150MT1, symbol BassingaLib_Inductors:ASPI-0628-3R9M-T1
- C191: value 100pF 100V -> 22uF 25V; footprint Capacitor_SMD:C_0603_1608Metric -> Capacitor_SMD:C_1210_3225Metric; Manufacturer_Part_Number CL10C101JC81PNC -> CL32B226KAJNNNE; Packaging 0603 (608mm) -> 1210 (3225mm)
Connections:
- net +3.3V_Digital: now also IC37.1 (FB), L2.2
- net +Vbus: now also IC37.2 (EN), IC37.3 (VIN)
- net GND: now also C191.1, IC37.4 (GND)
- net SW: no longer C144.1
- net at C144.2: now also IC37.6 (BST)
- new net: C144.1, IC37.5 (SW), L2.1
Other:
- moved on the sheet: LED10, LED11, LED12, R190, R193, R194

Commit message: Supervisor Block
Parts:
- TP6: renamed from TP3; footprint (none) -> TestPoint:TestPoint_Pad_D1.0mm
- renumbered C140 to C157, C139 to C158, C142 to C159, C144 to C160, C143 to C161, C146 to C162, C218 to C163, C219 to C164, C147 to C165, C148 to C166, C191 to C167, C149 to C168, C150 to C169, C192 to C170, C151 to C171, C152 to C172, C153 to C173, C154 to C174, C155 to C175, C156 to C176, C157 to C177, C158 to C178, C159 to C179, C160 to C180, D39 to D38, D48 to D39, IC37 to IC29, R243 to R189, R186 to R190, R187 to R191, R188 to R192, R189 to R193, R191 to R194, R192 to R195, R190 to R196, R193 to R197, R194 to R198, R195 to R199, R196 to R200, TP1 to TP4, TP2 to TP5

Commit message: Components library added
Parts:
- TP4, TP5, TP6: now left out of the parts list
Changed lines of the file:
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@@
 		(unit 1)
 		(exclude_from_sim no)
-		(in_bom yes)
+		(in_bom no)
 		(on_board yes)
 		(dnp no)
@@
 		(unit 1)
 		(exclude_from_sim no)
-		(in_bom yes)
+		(in_bom no)
 		(on_board yes)
 		(dnp no)
@@
 		(unit 1)
 		(exclude_from_sim no)
-		(in_bom yes)
+		(in_bom no)
 		(on_board yes)
 		(dnp no)

Commit message: Fly controller design started
Other:
- company: BASSINGA Lab -> BASSINGA_LAB
- title: (none) -> Propulsion Control Unit
Changed lines of the file:
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@@
 	(paper "A3")
 	(title_block
+		(title "Propulsion Control Unit")
 		(date "2025-05-21")
 		(rev "v1.0")
-		(company "BASSINGA Lab")
+		(company "BASSINGA_LAB")
+		(comment 1 "Copyright © 2025 Andresse Brisel BASSINGA ")
 	)
 	(rectangle
